Commit message: updated yaw angle of robotiqGripper

File: UR5e_with_2F_140_robotiq_gripper_RViz/universal_robot/ur_description/urdf/ur5e_robot.xacro (robot description, xacro)
@@ -21,5 +21,5 @@
   <!-- Define the joint connecting the wrist of the UR5e to the base link of the gripper -->
   <joint name="wrist_3_to_gripper_joint" type="fixed">
-    <origin xyz="0 0 0" rpy="0 0 0"/> <!-- Adjust as needed for correct positioning -->
+    <origin xyz="0 0 0" rpy="0 0 1.5707963267948966"/> <!-- Adjust as needed for correct positioning -->
     <parent link="wrist_3_link"/>
     <child link="robotiq_arg2f_base_link"/> <!-- Ensure this matches the actual base link name -->
