Commit message: scaling forearm colision with 1.005 to avoid the 2.8cm protective stop from teach pendant

File: UR5e_with_2F_140_robotiq_gripper_RViz/universal_robot/ur_description/urdf/ur5e_robot.urdf (robot description, URDF)
Before this commit: robot ur5e_robot, 22 links, 21 joints
Links:
- link forearm_link: geometry collision mesh filename=package://ur_description/meshes/ur5e/collision/forearm_test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; visual mesh filename=package://ur_description/meshes/ur5e/visual/forearm.dae
